Commit message: major: working simulation with minor bugs related to IMU data, working on those

File: rihibot_description/urdf/from_webots.urdf (robot description, URDF)
Before this commit: robot /home/diogo/catkin_ws/src/robots/rihibot/rihibot_description/urdf/ur10e.urdf, 11 links, 10 joints
Links:
- removed link hand_rgb_link
- removed link hand_rgb_optical_frame
Joints:
- removed joint hand_rgb_link_hand_rgb_optical_frame_joint
- removed joint wrist_3_link_hand_rgb_link_joint
- joint elbow_joint: origin xyz=0 -0.137 0.613 rpy=0 0 0 -> xyz=0 -0.137 0.613 rpy=0 -0.000135 0
- joint shoulder_lift_joint: origin xyz=0 0.176 0 rpy=0 1.570796 0 -> xyz=0 0.176 0 rpy=3.141593 1.570507 3.141593
- joint shoulder_pan_joint: origin xyz=0 0 0.181 rpy=0 0 0 -> xyz=0 0 0.181 rpy=0 0 -0.000174
- joint wrist_1_joint: origin xyz=0 0 0.571 rpy=0 1.570796 0 -> xyz=0 0 0.571 rpy=0 1.570794 0
- joint wrist_2_joint: origin xyz=0 0.135 0 rpy=0 0 0 -> xyz=0 0.135 0 rpy=0 0 -0.000011
- joint wrist_3_joint: origin xyz=0 0 0.12 rpy=0 0 0 -> xyz=0 0 0.12 rpy=0 -0.000019 0
