Commit message: fix: corrected camera links poses in urdf for robot_state_publisher

File: rihibot_description/urdf/compiled.urdf (robot description, URDF)
Before this commit: robot ur10e_robot, 15 links, 14 joints
Joints:
- joint tool0_hand_rgb_link_joint: origin xyz=0.0225 0.12 0 rpy=1.570793 0.000001 0 -> xyz=0 0 0 rpy=-1.5707963 -1.5707963 0

File: rihibot_description/urdf/from_webots.urdf (robot description, URDF)
Before this commit: robot /home/diogo/rihibot_ws/src/robots/rihibot/rihibot_description/urdf/from_webots.urdf, 9 links, 8 joints
Links:
- removed link accelerometer
- removed link forearm_link
- removed link gyro
- removed link shoulder_link
- removed link upper_arm_link
- removed link wrist_1_link
- removed link wrist_2_link
- removed link wrist_3_link
- added link camera
- link base_link: geometry 
Joints:
- removed joint elbow_joint
- removed joint shoulder_lift_joint
- removed joint shoulder_pan_joint
- removed joint wrist_1_joint
- removed joint wrist_2_joint
- removed joint wrist_3_joint
- removed joint wrist_3_link_accelerometer_joint
- removed joint wrist_3_link_gyro_joint
- added joint base_link_camera_joint: type fixed, parent base_link, child camera, origin xyz=0 0 0 rpy=0.063814 -1.570794 1.506984

File: rihibot_description/urdf/ur.xacro (robot description, xacro)
@@ -33,5 +33,5 @@
     <parent link="tool0"/>
     <child link="hand_rgb_link"/>
-    <origin rpy="1.570793 0.000001 0" xyz="0.0225 0.12 0"/>
+    <origin rpy="-${pi/2} -${pi/2} 0" xyz="0 0 0"/>
   </joint>
   <link name="hand_rgb_optical_frame">
