Commit message: minor: improved visualization in RViz

File: rihibot_description/urdf/UR10e_test.urdf (robot description, URDF)
Before this commit: robot /home/diogo/ros_workspaces/rihibot_ws/src/robots/rihibot/rihibot_description/urdf/UR10e_test.urdf, 10 links, 9 joints
Links:
- link accelerometer: geometry visual box size=0.02 0.02 0.02
- link base_link: geometry collision mesh filename=package://rihibot_description/meshes/ur10e/collision/base.s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; visual mesh filename=package://rihibot_description/meshes/ur10e/visual/base.dae
- link forearm_link: geometry collision mesh filename=package://rihibot_description/meshes/ur10e/collision/forear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; visual mesh filename=package://rihibot_description/meshes/ur10e/visual/forearm.d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
- link hand_rgb: geometry visual mesh filename=package://rihibot_description/meshes/rgb_camera/rgb_camera.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 scale=0.5 0.5 0.5
- link shoulder_link: geometry collision mesh filename=package://rihibot_description/meshes/ur10e/collision/should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; visual mesh filename=package://rihibot_description/meshes/ur10e/visual/shoulder.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
- link upper_arm_link: geometry collision mesh filename=package://rihibot_description/meshes/ur10e/collision/uppera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; visual mesh filename=package://rihibot_description/meshes/ur10e/visual/upperarm.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
- link wrist_1_link: geometry collision mesh filename=package://rihibot_description/meshes/ur10e/collision/wrist1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; visual mesh filename=package://rihibot_description/meshes/ur10e/visual/wrist1.dae
- link wrist_2_link: geometry collision mesh filename=package://rihibot_description/meshes/ur10e/collision/wrist2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; visual mesh filename=package://rihibot_description/meshes/ur10e/visual/wrist2.dae
- link wrist_3_link: geometry collision mesh filename=package://rihibot_description/meshes/ur10e/collision/wrist3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; visual mesh filename=package://rihibot_description/meshes/ur10e/visual/wrist3.dae
Joints:
- joint wrist_3_link_hand_rgb_joint: origin xyz=0 0.13 -0.02 rpy=1.570794 0.000002 0.000004 -> xyz=0 0.13 -0.02 rpy=-3.1415927 0 1.5707963
