Commit message: major: fixed simulation of rihibot (IMU only; missing camera)

File: rihibot_calibration/urdf/initial_estimate.urdf.xacro (robot description, xacro)
@@ -350,6 +350,6 @@
   <link name="hand_rgb_link">
 </link>
-  <joint name="wrist_3_link_hand_rgb_link_joint" type="fixed">
-    <parent link="wrist_3_link"/>
+  <joint name="tool0_hand_rgb_link_joint" type="fixed">
+    <parent link="tool0"/>
     <child link="hand_rgb_link"/>
     <origin rpy="1.570793 0.000001 0" xyz="0.0225 0.12 0"/>
@@ -364,15 +364,15 @@
   <link name="gyro">
 </link>
-  <joint name="wrist_3_link_gyro_joint" type="fixed">
-    <parent link="wrist_3_link"/>
+  <joint name="tool0_gyro_joint" type="fixed">
+    <parent link="tool0"/>
     <child link="gyro"/>
-    <origin rpy="3.141591 0.000002 1.570805" xyz="-0.0225 0.12 0"/>
+    <origin rpy="0 0 0" xyz="0 0 0"/>
   </joint>
   <link name="accelerometer">
 </link>
-  <joint name="wrist_3_link_accelerometer_joint" type="fixed">
-    <parent link="wrist_3_link"/>
+  <joint name="tool0_accelerometer_joint" type="fixed">
+    <parent link="tool0"/>
     <child link="accelerometer"/>
-    <origin rpy="3.141591 0.000002 1.570805" xyz="-0.0225 0.12 0"/>
+    <origin rpy="0 0 0" xyz="0 0 0"/>
   </joint>
 </robot>

File: rihibot_description/urdf/ur.xacro (robot description, xacro)
@@ -28,31 +28,31 @@
      safety_pos_margin="$(arg safety_pos_margin)"
      safety_k_position="$(arg safety_k_position)"/>
-<link name="hand_rgb_link">
+  <link name="hand_rgb_link">
 </link>
-<joint name="wrist_3_link_hand_rgb_link_joint" type="fixed">
-<parent link="wrist_3_link"/>
-<child link="hand_rgb_link"/>
-<origin xyz="0.0225 0.12 0" rpy="1.570793 0.000001 0"/>
-</joint>
-<link name="hand_rgb_optical_frame">
+  <joint name="tool0_hand_rgb_link_joint" type="fixed">
+    <parent link="tool0"/>
+    <child link="hand_rgb_link"/>
+    <origin rpy="1.570793 0.000001 0" xyz="0.0225 0.12 0"/>
+  </joint>
+  <link name="hand_rgb_optical_frame">
 </link>
-<joint name="hand_rgb_link_hand_rgb_optical_frame_joint" type="fixed">
-<parent link="hand_rgb_link"/>
-<child link="hand_rgb_optical_frame"/>
-<origin xyz="0 0 0" rpy="-1.570801 0.000006 -1.570798"/>
-</joint>
-<link name="gyro">
+  <joint name="hand_rgb_link_hand_rgb_optical_frame_joint" type="fixed">
+    <parent link="hand_rgb_link"/>
+    <child link="hand_rgb_optical_frame"/>
+    <origin rpy="-1.570801 0.000006 -1.570798" xyz="0 0 0"/>
+  </joint>
+  <link name="gyro">
 </link>
-<joint name="wrist_3_link_gyro_joint" type="fixed">
-<parent link="wrist_3_link"/>
-<child link="gyro"/>
-<origin xyz="-0.0225 0.12 0" rpy="3.141591 0.000002 1.570805"/>
-</joint>
-<link name="accelerometer">
+  <joint name="tool0_gyro_joint" type="fixed">
+    <parent link="tool0"/>
+    <child link="gyro"/>
+    <origin rpy="0 0 0" xyz="0 0 0"/>
+  </joint>
+  <link name="accelerometer">
 </link>
-<joint name="wrist_3_link_accelerometer_joint" type="fixed">
-<parent link="wrist_3_link"/>
-<child link="accelerometer"/>
-<origin xyz="-0.0225 0.12 0" rpy="3.141591 0.000002 1.570805"/>
-</joint>
+  <joint name="tool0_accelerometer_joint" type="fixed">
+    <parent link="tool0"/>
+    <child link="accelerometer"/>
+    <origin rpy="0 0 0" xyz="0 0 0"/>
+  </joint>
 </robot>

Commit message: minor: added camera visuals to URDF for RViz lardemua/atom#1026

File: rihibot_calibration/urdf/initial_estimate.urdf.xacro (robot description, xacro)
@@ -349,5 +349,14 @@
   </joint>
   <link name="hand_rgb_link">
-</link>
+    <visual>
+      <origin xyz="0.01 0 0" rpy="0 0 0" />
+      <geometry>
+        <mesh
+          filename="package://rihibot_description/meshes/rgb_camera/rgb_camera.stl"
+          scale="1 1 1" />
+      </geometry>
+      <!-- <xacro:insert_block name="color_rviz" /> -->
+    </visual>
+  </link>
   <joint name="tool0_hand_rgb_link_joint" type="fixed">
     <parent link="tool0"/>

File: rihibot_calibration/urdf/optimized.urdf.xacro (robot description, xacro)
@@ -301,5 +301,5 @@
   <link name="accelerometer"/>
   <joint name="tool0_accelerometer_joint" type="fixed">
-    <origin xyz="-0.014133962405914902 0.04218567218123059 -0.07632322268552906" rpy="0.0031500014025112187 0.000524009005636202 0.007370133530843516"/>
+    <origin xyz="0.04406709983384231 0.030022939246417114 0.0069761349108057764" rpy="0.0025215245161033825 0.00032166119894064125 -0.00033331493509894107"/>
     <parent link="tool0"/>
     <child link="accelerometer"/>

File: rihibot_calibration/urdf/optimized_w_pattern.urdf.xacro (robot description, xacro)
@@ -301,21 +301,7 @@
   <link name="accelerometer"/>
   <joint name="tool0_accelerometer_joint" type="fixed">
-    <origin xyz="-0.014133962405914902 0.04218567218123059 -0.07632322268552906" rpy="0.0031500014025112187 0.000524009005636202 0.007370133530843516"/>
+    <origin xyz="0.04406709983384231 0.030022939246417114 0.0069761349108057764" rpy="0.0025215245161033825 0.00032166119894064125 -0.00033331493509894107"/>
     <parent link="tool0"/>
     <child link="accelerometer"/>
   </joint>
-  <link name="pattern_link">
-    <origin xyz="0 0 0" rpy="0 0 0"/>
-    <visual name="pattern_1_visual">
-      <origin xyz="0 0 0" rpy="0 0 0"/>
-      <geometry>
-        <mesh filename="package://rihibot_webots/libraries/charuco_800x600_5x5_100/charuco_800x600_5x5_100.dae"/>
-      </geometry>
-    </visual>
-  </link>
-  <joint name="base_link-pattern_link" type="fixed">
-    <origin xyz="4.354556206922859 -0.44563768588970265 0.20442962080857002" rpy="1.3471669150188519 0.07936274168783991 1.813268210920521"/>
-    <parent link="base_link"/>
-    <child link="pattern_link"/>
-  </joint>
 </robot>

File: rihibot_description/urdf/ur.xacro (robot description, xacro)
@@ -29,5 +29,14 @@
      safety_k_position="$(arg safety_k_position)"/>
   <link name="hand_rgb_link">
-</link>
+    <visual>
+      <origin xyz="0.01 0 0" rpy="0 0 0" />
+      <geometry>
+        <mesh
+          filename="package://rihibot_description/meshes/rgb_camera/rgb_camera.stl"
+          scale="1 1 1" />
+      </geometry>
+      <!-- <xacro:insert_block name="color_rviz" /> -->
+    </visual>
+  </link>
   <joint name="tool0_hand_rgb_link_joint" type="fixed">
     <parent link="tool0"/>

Commit message: minor: added pattern to urdf for RViz lardemua/atom#1026

File: rihibot_calibration/urdf/initial_estimate.urdf.xacro (robot description, xacro)
@@ -385,3 +385,32 @@
     <origin rpy="0 0 0" xyz="0 0 0"/>
   </joint>
+<!-- chessboard link-->
+    <link name="chessboard_1200x900_10x7">
+        <visual>
+            <origin xyz="0 0 0" rpy="1.570801 0 0" />
+            <geometry>
+              <mesh filename="package://rihibot_webots/libraries/chessboard_1200x900_10x7/chessboard_1200x900_10x7.dae"
+                    scale="1 1 1" />
+            </geometry>
+            <!-- <material name="tripod_color" /> -->
+        </visual>
+        <collision name="tripod_collision">
+            <origin xyz="0 0 0" rpy="0 0 0" />
+            <geometry>
+              <mesh filename="package://rihibot_webots/libraries/chessboard_1200x900_10x7/chessboard_1200x900_10x7.dae"
+                    scale="1 1 1" />
+            </geometry>
+        </collision>
+        <inertial>
+            <mass value="1.0" />
+            <origin xyz="0 0 0" rpy="0 0 0" />
+            <inertia ixx="1" ixy="0" ixz="0" iyy="1" iyz="0" izz="1" />
+        </inertial>
+    </link>
+    <!-- tripod plate to tripod center support -->
+    <joint name="base_link_to_chessboard_1200x900_10x7" type="fixed">
+        <parent link="base_link" />
+        <child link="chessboard_1200x900_10x7"/>
+        <origin xyz="4.36168 -0.400363 0.27982 " rpy="-0.0000002 -0.2617985 1.8325937" />
+    </joint>
 </robot>

File: rihibot_description/urdf/ur.xacro (robot description, xacro)
@@ -65,3 +65,32 @@
     <origin rpy="0 0 0" xyz="0 0 0"/>
   </joint>
+  <!-- chessboard link-->
+    <link name="chessboard_1200x900_10x7">
+        <visual>
+          <origin xyz="0 0 0" rpy="${pi/2} 0 0" />
+            <geometry>
+              <mesh filename="package://rihibot_webots/libraries/chessboard_1200x900_10x7/chessboard_1200x900_10x7.dae"
+                    scale="1 1 1" />
+            </geometry>
+            <!-- <material name="tripod_color" /> -->
+        </visual>
+        <collision name="tripod_collision">
+            <origin xyz="0 0 0" rpy="0 0 0" />
+            <geometry>
+              <mesh filename="package://rihibot_webots/libraries/chessboard_1200x900_10x7/chessboard_1200x900_10x7.dae"
+                    scale="1 1 1" />
+            </geometry>
+        </collision>
+        <inertial>
+            <mass value="1.0" />
+            <origin xyz="0 0 0" rpy="0 0 0" />
+            <inertia ixx="1" ixy="0" ixz="0" iyy="1" iyz="0" izz="1" />
+        </inertial>
+    </link>
+    <!-- tripod plate to tripod center support -->
+    <joint name="base_link_to_chessboard_1200x900_10x7" type="fixed">
+        <parent link="base_link" />
+        <child link="chessboard_1200x900_10x7"/>
+        <origin xyz="4.36168 -0.400363 0.27982 " rpy="-0.0000002 -0.2617985 1.8325937" />
+    </joint>
 </robot>

Commit message: minor: added robotMover.py script - to be edited for testing lardemua/atom#1024

File: rihibot_calibration/urdf/initial_estimate.urdf.xacro (robot description, xacro)
@@ -321,5 +321,12 @@
     <parent link="wrist_3_link"/>
     <child link="accelerometer"/>
-    <origin xyz="0 0.13 0" rpy="0 0 0"/>
+    <origin xyz="0 0.13 0.02" rpy="0 0 0"/>
+  </joint>
+  <link name="hand_rgb">
+  </link>
+  <joint name="wrist_3_link_hand_rgb_joint" type="fixed">
+    <parent link="wrist_3_link"/>
+    <child link="hand_rgb"/>
+    <origin xyz="0 0.13 -0.02" rpy="1.570794 0.000002 0.000004"/>
   </joint>
 </robot>

Commit message: minor: updated urdf with correct gyro pose; improved joints movement for dataset lardemua/atom#1024

File: rihibot_calibration/urdf/initial_estimate.urdf.xacro (robot description, xacro)
@@ -314,5 +314,5 @@
     <parent link="wrist_3_link"/>
     <child link="gyro"/>
-    <origin xyz="0 0.13 0" rpy="0 0 0"/>
+    <origin xyz="0 0.13 0.02" rpy="0 0 0"/>
   </joint>
   <link name="accelerometer">

File: rihibot_calibration/urdf/optimized.urdf.xacro (robot description, xacro)
@@ -311,5 +311,5 @@
   <link name="gyro"/>
   <joint name="wrist_3_link_gyro_joint" type="fixed">
-    <origin xyz="0.0 0.13 0.0" rpy="0.0 0.0 0.0"/>
+    <origin xyz="0.0 0.13 0.02" rpy="0.0 0.0 0.0"/>
     <parent link="wrist_3_link"/>
     <child link="gyro"/>
@@ -317,7 +317,13 @@
   <link name="accelerometer"/>
   <joint name="wrist_3_link_accelerometer_joint" type="fixed">
-    <origin xyz="-0.16623351723058002 0.13850167432629829 0.040141947910749425" rpy="2.628944373253052e-06 -3.786397465896448e-05 -6.816176943571222e-05"/>
+    <origin xyz="0.0005263432993847853 0.13551521549650788 0.0016544206626573394" rpy="-0.00013378940826203883 -3.393275250867903e-05 0.00017693726214995607"/>
     <parent link="wrist_3_link"/>
     <child link="accelerometer"/>
   </joint>
+  <link name="hand_rgb"/>
+  <joint name="wrist_3_link_hand_rgb_joint" type="fixed">
+    <origin xyz="0.0 0.13 -0.02" rpy="1.570794 2e-06 4e-06"/>
+    <parent link="wrist_3_link"/>
+    <child link="hand_rgb"/>
+  </joint>
 </robot>
