Commit message: major(webots-ros): finished adapting the controllers to properly work with ROS lardemua/atom#1020

File: rihibot_calibration/urdf/optimized_w_pattern.urdf.xacro (robot description, xacro)
@@ -1,7 +1,7 @@
-<?xml version="1.0"?>
-<robot name="/home/diogo/catkin_ws/src/robots/rihibot/rihibot_description/urdf/ur5e.urdf" xmlns:xacro="http://ros.org/wiki/xacro">
+<?xml version="1.0" ?>
+<robot name="/home/diogo/catkin_ws/src/robots/rihibot/rihibot_description/urdf/ur5e.urdf" version="1.0">
   <link name="base_link">
     <visual>
-      <origin xyz="0 0 0.05" rpy="0 0 0"/>
+      <origin xyz="0.0 0.0 0.05" rpy="0.0 0.0 0.0"/>
       <geometry>
         <cylinder radius="0.076" length="0.1"/>
@@ -9,5 +9,5 @@
     </visual>
     <collision>
-      <origin xyz="0 0 0.05" rpy="0 0 0"/>
+      <origin xyz="0.0 0.0 0.05" rpy="0.0 0.0 0.0"/>
       <geometry>
         <cylinder radius="0.076" length="0.1"/>
@@ -16,13 +16,13 @@
   </link>
   <joint name="shoulder_pan_joint" type="revolute">
+    <origin xyz="0.0 0.0 0.163" rpy="0.0 0.0 0.0"/>
+    <axis xyz="0.0 0.0 1.0"/>
     <parent link="base_link"/>
     <child link="shoulder_link"/>
-    <axis xyz="0 0 1"/>
-    <limit effort="150" lower="-6.28319" upper="6.28319" velocity="3.14"/>
-    <origin xyz="0 0 0.163" rpy="0 0 0"/>
+    <limit effort="150.0" lower="-6.28319" upper="6.28319" velocity="3.14"/>
   </joint>
   <link name="shoulder_link">
     <visual>
-      <origin xyz="0 0 0" rpy="0 0 0"/>
+      <origin xyz="0.0 0.0 0.0" rpy="0.0 0.0 0.0"/>
       <geometry>
         <cylinder radius="0.059" length="0.135"/>
@@ -30,5 +30,5 @@
     </visual>
     <collision>
-      <origin xyz="0 0 0" rpy="0 0 0"/>
+      <origin xyz="0.0 0.0 0.0" rpy="0.0 0.0 0.0"/>
       <geometry>
         <cylinder radius="0.059" length="0.135"/>
@@ -36,5 +36,5 @@
     </collision>
     <visual>
-      <origin xyz="0 0.03 0" rpy="-1.570796 0 0"/>
+      <origin xyz="0.0 0.03 0.0" rpy="-1.570796 0.0 0.0"/>
       <geometry>
         <cylinder radius="0.059" length="0.093"/>
@@ -42,5 +42,5 @@
     </visual>
     <collision>
-      <origin xyz="0 0.03 0" rpy="-1.570796 0 0"/>
+      <origin xyz="0.0 0.03 0.0" rpy="-1.570796 0.0 0.0"/>
       <geometry>
         <cylinder radius="0.059" length="0.093"/>
@@ -49,13 +49,13 @@
   </link>
   <joint name="shoulder_lift_joint" type="revolute">
+    <origin xyz="0.0 0.138 0.0" rpy="0.0 1.570796 0.0"/>
+    <axis xyz="0.0 1.0 0.0"/>
     <parent link="shoulder_link"/>
     <child link="upper_arm_link"/>
-    <axis xyz="0 1 0"/>
-    <limit effort="150" lower="-6.28319" upper="6.28319" velocity="3.14"/>
-    <origin xyz="0 0.138 0" rpy="0 1.570796 0"/>
+    <limit effort="150.0" lower="-6.28319" upper="6.28319" velocity="3.14"/>
   </joint>
   <link name="upper_arm_link">
     <visual>
-      <origin xyz="0 0 0.22" rpy="0 0 0"/>
+      <origin xyz="0.0 0.0 0.22" rpy="0.0 0.0 0.0"/>
       <geometry>
         <cylinder radius="0.059" length="0.407"/>
@@ -63,5 +63,5 @@
     </visual>
     <collision>
-      <origin xyz="0 0 0.22" rpy="0 0 0"/>
+      <origin xyz="0.0 0.0 0.22" rpy="0.0 0.0 0.0"/>
       <geometry>
         <cylinder radius="0.059" length="0.407"/>
@@ -69,5 +69,5 @@
     </collision>
     <visual>
-      <origin xyz="0 0 0" rpy="-1.570796 0 0"/>
+      <origin xyz="0.0 0.0 0.0" rpy="-1.570796 0.0 0.0"/>
       <geometry>
         <cylinder radius="0.059" length="0.133"/>
@@ -75,5 +75,5 @@
     </visual>
     <collision>
-      <origin xyz="0 0 0" rpy="-1.570796 0 0"/>
+      <origin xyz="0.0 0.0 0.0" rpy="-1.570796 0.0 0.0"/>
       <geometry>
         <cylinder radius="0.059" length="0.133"/>
@@ -81,5 +81,5 @@
     </collision>
     <visual>
-      <origin xyz="0 -0.005 0.424" rpy="-1.570796 0 0"/>
+      <origin xyz="0.0 -0.005 0.424" rpy="-1.570796 0.0 0.0"/>
       <geometry>
         <cylinder radius="0.059" length="0.149"/>
@@ -87,5 +87,5 @@
     </visual>
     <collision>
-      <origin xyz="0 -0.005 0.424" rpy="-1.570796 0 0"/>
+      <origin xyz="0.0 -0.005 0.424" rpy="-1.570796 0.0 0.0"/>
       <geometry>
         <cylinder radius="0.059" length="0.149"/>
@@ -94,13 +94,13 @@
   </link>
   <joint name="elbow_joint" type="revolute">
+    <origin xyz="0.0 -0.131 0.425" rpy="0.0 0.0 0.0"/>
+    <axis xyz="0.0 1.0 0.0"/>
     <parent link="upper_arm_link"/>
     <child link="forearm_link"/>
-    <axis xyz="0 1 0"/>
-    <limit effort="150" lower="-3.14159" upper="3.14159" velocity="3.14"/>
-    <origin xyz="0 -0.131 0.425" rpy="0 0 0"/>
+    <limit effort="150.0" lower="-3.14159" upper="3.14159" velocity="3.14"/>
   </joint>
   <link name="forearm_link">
     <visual>
-      <origin xyz="0 0 0.207" rpy="0 0 0"/>
+      <origin xyz="0.0 0.0 0.207" rpy="0.0 0.0 0.0"/>
       <geometry>
         <cylinder radius="0.038" length="0.36"/>
@@ -108,5 +108,5 @@
     </visual>
     <collision>
-      <origin xyz="0 0 0.207" rpy="0 0 0"/>
+      <origin xyz="0.0 0.0 0.207" rpy="0.0 0.0 0.0"/>
       <geometry>
         <cylinder radius="0.038" length="0.36"/>
@@ -114,5 +114,5 @@
     </collision>
     <visual>
-      <origin xyz="0 -0.001 0.39" rpy="-1.570796 0 0"/>
+      <origin xyz="0.0 -0.001 0.39" rpy="-1.570796 0.0 0.0"/>
       <geometry>
         <cylinder radius="0.039" length="0.109"/>
@@ -120,5 +120,5 @@
     </visual>
     <collision>
-      <origin xyz="0 -0.001 0.39" rpy="-1.570796 0 0"/>
+      <origin xyz="0.0 -0.001 0.39" rpy="-1.570796 0.0 0.0"/>
       <geometry>
         <cylinder radius="0.039" length="0.109"/>
@@ -126,5 +126,5 @@
     </collision>
     <visual>
-      <origin xyz="0 0.06 0" rpy="1.570796 0 0"/>
+      <origin xyz="0.0 0.06 0.0" rpy="1.570796 0.0 0.0"/>
       <geometry>
         <cylinder radius="0.058" length="0.05"/>
@@ -132,5 +132,5 @@
     </visual>
     <collision>
-      <origin xyz="0 0.06 0" rpy="1.570796 0 0"/>
+      <origin xyz="0.0 0.06 0.0" rpy="1.570796 0.0 0.0"/>
       <geometry>
         <cylinder radius="0.058" length="0.05"/>
@@ -138,5 +138,5 @@
     </collision>
     <visual>
-      <origin xyz="0 0.06 0.025" rpy="1.570796 0 0"/>
+      <origin xyz="0.0 0.06 0.025" rpy="1.570796 0.0 0.0"/>
       <geometry>
         <sphere radius="0.058"/>
@@ -144,5 +144,5 @@
     </visual>
     <collision>
-      <origin xyz="0 0.06 0.025" rpy="1.570796 0 0"/>
+      <origin xyz="0.0 0.06 0.025" rpy="1.570796 0.0 0.0"/>
       <geometry>
         <sphere radius="0.058"/>
@@ -150,5 +150,5 @@
     </collision>
     <visual>
-      <origin xyz="0 0.06 -0.025" rpy="1.570796 0 0"/>
+      <origin xyz="0.0 0.06 -0.025" rpy="1.570796 0.0 0.0"/>
       <geometry>
         <sphere radius="0.058"/>
@@ -156,5 +156,5 @@
     </visual>
     <collision>
-      <origin xyz="0 0.06 -0.025" rpy="1.570796 0 0"/>
+      <origin xyz="0.0 0.06 -0.025" rpy="1.570796 0.0 0.0"/>
       <geometry>
         <sphere radius="0.058"/>
@@ -162,5 +162,5 @@
     </collision>
     <visual>
-      <origin xyz="0 0 0.07" rpy="0 0 0"/>
+      <origin xyz="0.0 0.0 0.07" rpy="0.0 0.0 0.0"/>
       <geometry>
         <cylinder radius="0.04" length="0.1"/>
@@ -168,5 +168,5 @@
     </visual>
     <collision>
-      <origin xyz="0 0 0.07" rpy="0 0 0"/>
+      <origin xyz="0.0 0.0 0.07" rpy="0.0 0.0 0.0"/>
       <geometry>
         <cylinder radius="0.04" length="0.1"/>
@@ -174,5 +174,5 @@
     </collision>
     <visual>
-      <origin xyz="0 0.05 0.07" rpy="0 0 0"/>
+      <origin xyz="0.0 0.05 0.07" rpy="0.0 0.0 0.0"/>
       <geometry>
         <sphere radius="0.04"/>
@@ -180,5 +180,5 @@
     </visual>
     <collision>
-      <origin xyz="0 0.05 0.07" rpy="0 0 0"/>
+      <origin xyz="0.0 0.05 0.07" rpy="0.0 0.0 0.0"/>
       <geometry>
         <sphere radius="0.04"/>
@@ -186,5 +186,5 @@
     </collision>
     <visual>
-      <origin xyz="0 -0.05 0.07" rpy="0 0 0"/>
+      <origin xyz="0.0 -0.05 0.07" rpy="0.0 0.0 0.0"/>
       <geometry>
         <sphere radius="0.04"/>
@@ -192,5 +192,5 @@
     </visual>
     <collision>
-      <origin xyz="0 -0.05 0.07" rpy="0 0 0"/>
+      <origin xyz="0.0 -0.05 0.07" rpy="0.0 0.0 0.0"/>
       <geometry>
         <sphere radius="0.04"/>
@@ -199,13 +199,13 @@
   </link>
   <joint name="wrist_1_joint" type="revolute">
+    <origin xyz="0.0 0.0 0.392" rpy="0.0 1.570796 0.0"/>
+    <axis xyz="0.0 1.0 0.0"/>
     <parent link="forearm_link"/>
     <child link="wrist_1_link"/>
-    <axis xyz="0 1 0"/>
-    <limit effort="28" lower="-6.28319" upper="6.28319" velocity="6.28"/>
-    <origin xyz="0 0 0.392" rpy="0 1.570796 0"/>
+    <limit effort="28.0" lower="-6.28319" upper="6.28319" velocity="6.28"/>
   </joint>
   <link name="wrist_1_link">
     <visual>
-      <origin xyz="0 0.089 0" rpy="-1.570796 0 0"/>
+      <origin xyz="0.0 0.089 0.0" rpy="-1.570796 0.0 0.0"/>
       <geometry>
         <cylinder radius="0.038" length="0.086"/>
@@ -213,5 +213,5 @@
     </visual>
     <collision>
-      <origin xyz="0 0.089 0" rpy="-1.570796 0 0"/>
+      <origin xyz="0.0 0.089 0.0" rpy="-1.570796 0.0 0.0"/>
       <geometry>
         <cylinder radius="0.038" length="0.086"/>
@@ -219,5 +219,5 @@
     </collision>
     <visual>
-      <origin xyz="0 0.126 0" rpy="0 0 0"/>
+      <origin xyz="0.0 0.126 0.0" rpy="0.0 0.0 0.0"/>
       <geometry>
         <cylinder radius="0.038" length="0.112"/>
@@ -225,5 +225,5 @@
     </visual>
     <collision>
-      <origin xyz="0 0.126 0" rpy="0 0 0"/>
+      <origin xyz="0.0 0.126 0.0" rpy="0.0 0.0 0.0"/>
       <geometry>
         <cylinder radius="0.038" length="0.112"/>
@@ -232,13 +232,13 @@
   </link>
   <joint name="wrist_2_joint" type="revolute">
+    <origin xyz="0.0 0.127 0.0" rpy="0.0 0.0 0.0"/>
+    <axis xyz="0.0 0.0 1.0"/>
     <parent link="wrist_1_link"/>
     <child link="wrist_2_link"/>
-    <axis xyz="0 0 1"/>
-    <limit effort="28" lower="-6.28319" upper="6.28319" velocity="6.28"/>
-    <origin xyz="0 0.127 0" rpy="0 0 0"/>
+    <limit effort="28.0" lower="-6.28319" upper="6.28319" velocity="6.28"/>
   </joint>
   <link name="wrist_2_link">
     <visual>
-      <origin xyz="0 -0.001 0.0995" rpy="-1.570796 0 0"/>
+      <origin xyz="0.0 -0.001 0.0995" rpy="-1.570796 0.0 0.0"/>
       <geometry>
         <cylinder radius="0.04" length="0.108"/>
@@ -246,5 +246,5 @@
     </visual>
     <collision>
-      <origin xyz="0 -0.001 0.0995" rpy="-1.570796 0 0"/>
+      <origin xyz="0.0 -0.001 0.0995" rpy="-1.570796 0.0 0.0"/>
       <geometry>
         <cylinder radius="0.04" length="0.108"/>
@@ -252,5 +252,5 @@
     </collision>
     <visual>
-      <origin xyz="0 -0.001 0.0676" rpy="0 0 0"/>
+      <origin xyz="0.0 -0.001 0.0676" rpy="0.0 0.0 0.0"/>
       <geometry>
         <cylinder radius="0.038" length="0.043"/>
@@ -258,5 +258,5 @@
     </visual>
     <collision>
-      <origin xyz="0 -0.001 0.0676" rpy="0 0 0"/>
+      <origin xyz="0.0 -0.001 0.0676" rpy="0.0 0.0 0.0"/>
       <geometry>
         <cylinder radius="0.038" length="0.043"/>
@@ -265,13 +265,13 @@
   </link>
   <joint name="wrist_3_joint" type="revolute">
+    <origin xyz="0.0 0.0 0.1" rpy="0.0 0.0 0.0"/>
+    <axis xyz="0.0 1.0 0.0"/>
     <parent link="wrist_2_link"/>
     <child link="wrist_3_link"/>
-    <axis xyz="0 1 0"/>
-    <limit effort="28" lower="-6.28319" upper="6.28319" velocity="6.28"/>
-    <origin xyz="0 0 0.1" rpy="0 0 0"/>
+    <limit effort="28.0" lower="-6.28319" upper="6.28319" velocity="6.28"/>
   </joint>
   <link name="wrist_3_link">
     <visual>
-      <origin xyz="0 0.07 0" rpy="-1.570796 0 0"/>
+      <origin xyz="0.0 0.07 0.0" rpy="-1.570796 0.0 0.0"/>
       <geometry>
         <cylinder radius="0.038" length="0.048"/>
@@ -279,5 +279,5 @@
     </visual>
     <collision>
-      <origin xyz="0 0.07 0" rpy="-1.570796 0 0"/>
+      <origin xyz="0.0 0.07 0.0" rpy="-1.570796 0.0 0.0"/>
       <geometry>
         <cylinder radius="0.038" length="0.048"/>
@@ -285,5 +285,5 @@
     </collision>
     <visual>
-      <origin xyz="0 0.09 0" rpy="-1.570796 0 0"/>
+      <origin xyz="0.0 0.09 0.0" rpy="-1.570796 0.0 0.0"/>
       <geometry>
         <cylinder radius="0.032" length="0.018"/>
@@ -291,5 +291,5 @@
     </visual>
     <collision>
-      <origin xyz="0 0.09 0" rpy="-1.570796 0 0"/>
+      <origin xyz="0.0 0.09 0.0" rpy="-1.570796 0.0 0.0"/>
       <geometry>
         <cylinder radius="0.032" length="0.018"/>
@@ -297,31 +297,41 @@
     </collision>
   </link>
-  <link name="hand_rgb_link">
-  </link>
+  <link name="hand_rgb_link"/>
   <joint name="wrist_3_link_hand_rgb_link_joint" type="fixed">
+    <origin xyz="0.0225 0.1 0.0" rpy="1.570793 1e-06 0.0"/>
     <parent link="wrist_3_link"/>
     <child link="hand_rgb_link"/>
-    <origin xyz="0.0225 0.1 0" rpy="1.570793 0.000001 0"/>
-  </joint>
-  <link name="hand_rgb_optical_frame">
-  </link>
+  </joint>
+  <link name="hand_rgb_optical_frame"/>
   <joint name="hand_rgb_link_hand_rgb_optical_frame_joint" type="fixed">
+    <origin xyz="0.0 0.0 0.0" rpy="-1.570801 6e-06 -1.570798"/>
     <parent link="hand_rgb_link"/>
     <child link="hand_rgb_optical_frame"/>
-    <origin xyz="0 0 0" rpy="-1.570801 0.000006 -1.570798"/>
-  </joint>
-  <link name="accelerometer">
-  </link>
+  </joint>
+  <link name="accelerometer"/>
   <joint name="wrist_3_link_accelerometer_joint" type="fixed">
+    <origin xyz="0.1404272748964973 4.659850956736325 0.10128322305971679" rpy="3.1386331910351335 -0.00012576277697928963 1.566339794306187"/>
     <parent link="wrist_3_link"/>
     <child link="accelerometer"/>
-    <origin xyz="-0.0225 0.1 0" rpy="3.141591 0.000002 1.570805"/>
-  </joint>
-  <link name="gyro">
-  </link>
+  </joint>
+  <link name="gyro"/>
   <joint name="wrist_3_link_gyro_joint" type="fixed">
+    <origin xyz="-0.0225 0.1 0.0" rpy="3.141591 2e-06 1.570805"/>
     <parent link="wrist_3_link"/>
     <child link="gyro"/>
-    <origin xyz="-0.0225 0.1 0" rpy="3.141591 0.000002 1.570805"/>
+  </joint>
+  <link name="pattern_link">
+    <origin xyz="0 0 0" rpy="0 0 0"/>
+    <visual name="pattern_1_visual">
+      <origin xyz="0 0 0" rpy="0 0 0"/>
+      <geometry>
+        <mesh filename="package://rihibot_webots/libraries/charuco_800x600_5x5_100/charuco_800x600_5x5_100.dae"/>
+      </geometry>
+    </visual>
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
File: rihibot_description/urdf/ur5e.urdf (robot description, URDF)
Before this commit: robot /home/diogo/catkin_ws/src/robots/rihibot/rihibot_description/urdf/ur5e.urdf, 11 links, 10 joints
Joints:
- joint hand_rgb_link_hand_rgb_optical_frame_joint: origin xyz=0 0 0 rpy=-3.141595 0.000001 -3.141592 -> xyz=0 0 0 rpy=-1.570801 0.000006 -1.570798
- joint wrist_3_link_hand_rgb_link_joint: origin xyz=0.0225 0.1 0 rpy=-3.141587 -0.000005 1.570795 -> xyz=0.0225 0.1 0 rpy=1.570793 0.000001 0

Commit message: minor: added world with chessboard for compatibility with alternate calib methods

File: rihibot_calibration/urdf/optimized.urdf.xacro (robot description, xacro)
@@ -283,5 +283,5 @@
   <link name="hand_rgb_link"/>
   <joint name="tool0_hand_rgb_link_joint" type="fixed">
-    <origin xyz="0.0225 0.12 0.0" rpy="1.570793 1e-06 0.0"/>
+    <origin xyz="0.0 0.0 0.0" rpy="-1.5707963 -1.5707963 0.0"/>
     <parent link="tool0"/>
     <child link="hand_rgb_link"/>
@@ -301,5 +301,5 @@
   <link name="accelerometer"/>
   <joint name="tool0_accelerometer_joint" type="fixed">
-    <origin xyz="-0.017516383748223945 -0.011142495796901712 -0.00902252789045713" rpy="0.0002665379331080773 0.004899270832039293 -0.0030877532323734507"/>
+    <origin xyz="-0.014133962405914902 0.04218567218123059 -0.07632322268552906" rpy="0.0031500014025112187 0.000524009005636202 0.007370133530843516"/>
     <parent link="tool0"/>
     <child link="accelerometer"/>

File: rihibot_calibration/urdf/optimized_w_pattern.urdf.xacro (robot description, xacro)
@@ -283,5 +283,5 @@
   <link name="hand_rgb_link"/>
   <joint name="tool0_hand_rgb_link_joint" type="fixed">
-    <origin xyz="0.0225 0.12 0.0" rpy="1.570793 1e-06 0.0"/>
+    <origin xyz="0.0 0.0 0.0" rpy="-1.5707963 -1.5707963 0.0"/>
     <parent link="tool0"/>
     <child link="hand_rgb_link"/>
@@ -301,7 +301,21 @@
   <link name="accelerometer"/>
   <joint name="tool0_accelerometer_joint" type="fixed">
-    <origin xyz="-0.017516383748223945 -0.011142495796901712 -0.00902252789045713" rpy="0.0002665379331080773 0.004899270832039293 -0.0030877532323734507"/>
+    <origin xyz="-0.014133962405914902 0.04218567218123059 -0.07632322268552906" rpy="0.0031500014025112187 0.000524009005636202 0.007370133530843516"/>
     <parent link="tool0"/>
     <child link="accelerometer"/>
   </joint>
+  <link name="pattern_link">
+    <origin xyz="0 0 0" rpy="0 0 0"/>
+    <visual name="pattern_1_visual">
+      <origin xyz="0 0 0" rpy="0 0 0"/>
+      <geometry>
+        <mesh filename="package://rihibot_webots/libraries/charuco_800x600_5x5_100/charuco_800x600_5x5_100.dae"/>
+      </geometry>
+    </visual>
+  </link>
+  <joint name="base_link-pattern_link" type="fixed">
+    <origin xyz="4.354556206922859 -0.44563768588970265 0.20442962080857002" rpy="1.3471669150188519 0.07936274168783991 1.813268210920521"/>
+    <parent link="base_link"/>
+    <child link="pattern_link"/>
+  </joint>
 </robot>
